Commit message: rrt vis added

File: eufs_description/sensors/VLP-16.urdf.xacro (robot description, xacro)
@@ -2,5 +2,5 @@
 <robot xmlns:xacro="http://www.ros.org/wiki/xacro" name="VLP-16">
   <xacro:property name="M_PI" value="3.1415926535897931" />
-  <xacro:macro name="VLP-16" params="*origin parent:=base_link name:=velodyne topic:=/velodyne_points hz:=10 lasers:=16 samples:=1875 collision_range:=0.3 min_range:=0.9 max_range:=130.0 noise:=0.008 min_angle:=-${M_PI} max_angle:=${M_PI}">
+  <xacro:macro name="VLP-16" params="*origin parent:=base_link name:=velodyne topic:=/velodyne_points hz:=10 lasers:=16 samples:=1875 collision_range:=0.3 min_range:=0.9 max_range:=130.0 noise:=0.008 min_angle:=-${M_PI}/2 max_angle:=${M_PI}/2">
     <joint name="${name}_base_mount_joint" type="fixed">
       <xacro:insert_block name="origin" />

File: eufs_description/sensors/VLP-16R.urdf.xacro (robot description, xacro)
@@ -2,5 +2,5 @@
 <robot xmlns:xacro="http://www.ros.org/wiki/xacro" name="VLP-16">
   <xacro:property name="M_PI" value="3.1415926535897931" />
-  <xacro:macro name="VLP-16R" params="*origin parent:=base_link name:=velodyne topic:=/velodyne_points hz:=6 lasers:=5 samples:=1200 collision_range:=0.3 min_range:=0.6 max_range:=130.0 noise:=0.008 min_angle:=-2 max_angle:=2">
+  <xacro:macro name="VLP-16R" params="*origin parent:=base_link name:=velodyne topic:=/velodyne_points hz:=6 lasers:=5 samples:=1200 collision_range:=0.3 min_range:=0.6 max_range:=130.0 noise:=0.008 min_angle:=-1.57 max_angle:=1.57">
     <joint name="${name}_base_mount_joint" type="fixed">
       <xacro:insert_block name="origin" />
